File: converters.kicad_sch (KiCad schematic)
At the start: 22 parts, among them J1 USB_C_Receptacle, J2 DC 5V In, Q1 MMBT2222A-TP, U1 AP2112K-1.8, U2 TPS62160DSG

Commit message: Rev1 final commit
Connections:
- net 5_3V3_FB renamed 5_+3V3_FB
- net 5_3V3_SW renamed 5_+3V3_SW
Other:
- note added: "+3V3 to 1V8"
- note added: "5V to +3V3"
- note added: "R5 = 100k R4 = 100k((+3V3/0.8V) - 1) = 312.5k. USE 312k R3 = 100k, from datasheet"
- note removed: "3V3 to 1V8"
- note removed: "5V to 3V3"
- note removed: "R5 = 100k R4 = 100k((3V3/0.8V) - 1) = 312.5k. USE 312k R3 = 100k, from datasheet"
Changed lines of the file:
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@@
 		)
 	)
-	(text "3V3 to 1V8"
+	(text "+3V3 to 1V8"
 		(exclude_from_sim no)
 		(at 115.316 111.252 0)
@@
 		)
 	)
-	(text "R5 = 100k\nR4 = 100k((3V3/0.8V) - 1) = 312.5k. USE 312k\nR3 = 100k, from datasheet"
+	(text "R5 = 100k\nR4 = 100k((+3V3/0.8V) - 1) = 312.5k. USE 312k\nR3 = 100k, from datasheet"
 		(exclude_from_sim no)
 		(at 111.76 83.566 0)
@@
 		)
 	)
-	(text "5V to 3V3"
+	(text "5V to +3V3"
 		(exclude_from_sim no)
 		(at 117.602 42.418 0)
@@
 	)
 	(junction
-		(at 189.23 53.34)
-		(diameter 0)
-		(color 0 0 0 0)
-	)
-	(junction
 		(at 151.13 124.46)
 		(diameter 0)
@@
 	(wire
 		(pts
-			(xy 184.15 53.34) (xy 189.23 53.34)
-		)
-		(stroke
-			(width 0)
-			(type default)
-		)
-	)
-	(wire
-		(pts
 			(xy 19.05 184.15) (xy 19.05 187.96)
 		)
@@
 	(wire
 		(pts
-			(xy 189.23 53.34) (xy 194.31 53.34)
-		)
-		(stroke
-			(width 0)
-			(type default)
-		)
-	)
-	(wire
-		(pts
 			(xy 62.23 27.94) (xy 59.69 27.94)
 		)
@@
 	(wire
 		(pts
-			(xy 194.31 53.34) (xy 194.31 50.8)
-		)
-		(stroke
-			(width 0)
-			(type default)
-		)
-	)
-	(wire
-		(pts
 			(xy 140.97 134.62) (xy 140.97 137.16)
 		)
@@
 	(wire
 		(pts
-			(xy 189.23 53.34) (xy 189.23 44.45)
-		)
-		(stroke
-			(width 0)
-			(type default)
-		)
-	)
-	(wire
-		(pts
 			(xy 173.99 63.5) (xy 173.99 62.23)
 		)
@@
 		)
 	)
-	(label "5_3V3_VOS"
+	(label "5_+3V3_VOS"
 		(at 152.4 55.88 0)
 		(effects
@@
 		)
 	)
-	(label "5_3V3_PG"
+	(label "5_+3V3_PG"
 		(at 161.29 60.96 0)
 		(effects
@@
 		)
 	)
-	(label "5_3V3_FB"
+	(label "5_+3V3_FB"
 		(at 161.29 63.5 0)
 		(effects
@@
 		)
 	)
-	(label "5_3V3_SW"
+	(label "5_+3V3_SW"
 		(at 152.4 53.34 0)
 		(effects
@@
 	)
 	(symbol
-		(lib_id "power:+3V3")
-		(at 194.31 50.8 0)
-		(unit 1)
-		(body_style 1)
-		(exclude_from_sim no)
-		(in_bom yes)
-		(on_board yes)
-		(in_pos_files yes)
-		(dnp no)
-		(fields_autoplaced yes)
-		(property "Reference" "#PWR022"
-			(at 194.31 54.61 0)
-			(hide yes)
-			(show_name no)
-			(do_not_autoplace no)
-			(effects
-				(font
-					(size 1.27 1.27)
-				)
-			)
-		)
-		(property "Value" "MCU_VDDA"
-			(at 194.31 45.72 0)
-			(show_name no)
-			(do_not_autoplace no)
-			(effects
-				(font
-					(size 1.27 1.27)
-				)
-			)
-		)
-		(property "Footprint" ""
-			(at 194.31 50.8 0)
-			(hide yes)
-			(show_name no)
-			(do_not_autoplace no)
-			(effects
-				(font
-					(size 1.27 1.27)
-				)
-			)
-		)
-		(property "Datasheet" ""
-			(at 194.31 50.8 0)
-			(hide yes)
-			(show_name no)
-			(do_not_autoplace no)
-			(effects
-				(font
-					(size 1.27 1.27)
-				)
-			)
-		)
-		(property "Description" "Power symbol creates a global label with name \"+3V3\""
-			(at 194.31 50.8 0)
-			(hide yes)
-			(show_name no)
-			(do_not_autoplace no)
-			(effects
-				(font
-					(size 1.27 1.27)
-				)
-			)
-		)
-		(pin "1"
-		)
-		(instances
-			(project "Telemetry Box"
-				(path "/71a96c1a-3810-48e8-8b77-829a22b612db/e1044467-df55-4773-adfc-6bc275c0743b"
-					(reference "#PWR022")
-					(unit 1)
-				)
-			)
-		)
-	)
-	(symbol
 		(lib_id "power:Earth")
 		(at 52.07 130.81 0)
@@
 					(unit 1)
 				)
-			)
-		)
-	)
-	(symbol
-		(lib_id "power:+3V3")
-		(at 189.23 44.45 0)
-		(unit 1)
-		(body_style 1)
-		(exclude_from_sim no)
-		(in_bom yes)
-		(on_board yes)
-		(in_pos_files yes)
-		(dnp no)
-		(fields_autoplaced yes)
-		(property "Reference" "#PWR021"
-			(at 189.23 48.26 0)
-			(hide yes)
-			(show_name no)
-			(do_not_autoplace no)
-			(effects
-				(font
-					(size 1.27 1.27)
-				)
-			)
-		)
-		(property "Value" "MCU_VDD"
-			(at 189.23 39.37 0)
-			(show_name no)
-			(do_not_autoplace no)
-			(effects
-				(font
-					(size 1.27 1.27)
-				)
-			)
-		)
-		(property "Footprint" ""
-			(at 189.23 44.45 0)
-			(hide yes)
-			(show_name no)
-			(do_not_autoplace no)
-			(effects
-				(font
-					(size 1.27 1.27)
-				)
-			)
-		)
-		(property "Datasheet" ""
-			(at 189.23 44.45 0)
-			(hide yes)
-			(show_name no)
-			(do_not_autoplace no)
-			(effects
-				(font
-					(size 1.27 1.27)
-				)
-			)
-		)
-		(property "Description" "Power symbol creates a global label with name \"+3V3\""
-			(at 189.23 44.45 0)
-			(hide yes)
-			(show_name no)
-			(do_not_autoplace no)
-			(effects
-				(font
-					(size 1.27 1.27)
-				)
-			)
-		)
-		(pin "1"
-		)
-		(instances
-			(project "Telemetry Box"
-				(path "/71a96c1a-3810-48e8-8b77-829a22b612db/e1044467-df55-4773-adfc-6bc275c0743b"
-					(reference "#PWR021")
-					(unit 1)
-				)
