File: telem_mcu.kicad_sch (KiCad schematic)
At the start: 22 parts, among them J3 Conn_01x06, J5 Micro_SD_Card, SW2 SW_Push, SW3 SW_SPDT, U3 STM32F373CCTx, X1 32.768kHz

Commit message: Updated schematics for rev2
Parts:
- removed SW3: SW_SPDT, Telem_fp:SWITCH_1SCQN, symbol Switch:SW_SPDT
- added C18: 100nF, Capacitor_SMD:C_0603_1608Metric, symbol Device:C
- added R10, R11, R12, R13, R14, R8: 2k2, Resistor_SMD:R_0603_1608Metric, symbol Device:R_US
- C12, C17: footprint Capacitor_SMD:C_0805_2012Metric -> Capacitor_SMD:C_0603_1608Metric
- J5: footprint Connector_Card:microSD_HC_Molex_47219-2001 -> Telem_fp:AMPHENOL_10067099-200LF
Connections:
- net IMU_INT is gone; now on net THERM1_ADC: U3.18 (PB0)
- net MCU_VDD is gone; now on net +3V3: C5.1, C7.1, C9.1, J3.1 (Pin_1), U3.1 (VBAT), U3.17 (VDD), U3.48 (VDD)
- net MCU_VDDA is gone; now on net +3V3: C10.1, C11.1, C6.1, C8.1, U3.24 (VDDSD), U3.25 (VREFSD+), U3.9 (VDDA)
- net BMP_SCX: now also U3.45 (PB8), R11.1; no longer U3.42 (PB6)
- net BMP_SDX: now also U3.46 (PB9), R12.1; no longer U3.43 (PB7)
- net GPS_RST: now also U3.28 (PD8); no longer U3.41 (PB5)
- net GPS_SCL: now also R8.1
- net GPS_SDA: now also R10.1
- net GPS_TP: now also U3.29 (PA8); no longer U3.19 (PB1)
- net IMU_CS: now also U3.38 (PA15), R13.1; no longer U3.14 (PA4)
- net IMU_SDI: now also U3.41 (PB5); no longer U3.29 (PA8)
- net IMU_SDO: now also U3.40 (PB4); no longer U3.16 (PA6)
- net IMU_SPC: now also U3.39 (PB3); no longer U3.15 (PA5)
- net PGND: now also J5.6 (VSS), J5.SH (SHIELD), R15.1, C18.2
- net THERM1_ADC: no longer U3.10 (PA0)
- net THERM2_ADC: now also U3.16 (PA6); no longer U3.11 (PA1)
- net SD_CS: now reaches J5.2 (DAT3/CD)
- net SD_CS: now also U3.10 (PA0), R14.1
- net SD_MOSI: now reaches J5.3 (CMD)
- net SD_MOSI: now also U3.13 (PA3)
- net +3V3: now reaches J5.4 (VDD)
- net +3V3: now also C18.1, R10.2, R11.2, R12.2, R13.2, R14.2, R8.2
- net SD_CLK: now reaches J5.5 (CLK)
- net SD_CLK: now also U3.11 (PA1)
- net SD_MISO: now reaches J5.7 (DAT0)
- net SD_MISO: now also U3.12 (PA2)
- net Crystal_1: now reaches C15.2, U3.3 (PC14), X1.2
- net USB_DN: now reaches U3.32 (PA11)
- net USB_DP: now reaches U3.33 (PA12)
- net Crystal_2: now reaches C16.2, R9.1, X1.1
- no-connect marks 20 -> 18
Other:
- note added: "NRST Circuit"
- note added: "Pullup Resistors"
- note removed: "NRST and BOOT Circuits"
- moved on the sheet: C15, C16, C20, J5, R15, R9, SW2, X1

Commit message: Updated schematics for rev2
Other:
- note added: "Micro SD"
- moved on the sheet: C15, C16, C18, J5, R15, R9, U3, X1

Commit message: Initial Layout Rev2
Connections:
- net GPS_RST: now also U3.21 (PE8); no longer U3.28 (PD8)
- net GPS_TP: now also U3.22 (PE9); no longer U3.29 (PA8)
- net THERM1_ADC: now also U3.16 (PA6); no longer U3.18 (PB0)
- net THERM2_ADC: now also U3.18 (PB0); no longer U3.16 (PA6)
- no-connect marks 18 -> 15
Changed lines of the file:
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@@
-	)
-	(no_connect
-		(at 135.89 74.93)
-	)
-	(no_connect
-		(at 176.53 92.71)
 	)
 	(no_connect
@@
 		(at 135.89 69.85)
 	)
-	(no_connect
-		(at 135.89 77.47)
-	)
 	(wire
 		(pts
@@
 	(wire
 		(pts
-			(xy 132.08 82.55) (xy 135.89 82.55)
-		)
-		(stroke
-			(width 0)
-			(type default)
-		)
-	)
-	(wire
-		(pts
 			(xy 176.53 49.53) (xy 185.42 49.53)
 		)
@@
 	(wire
 		(pts
-			(xy 176.53 64.77) (xy 177.8 64.77)
-		)
-		(stroke
-			(width 0)
-			(type default)
-		)
-	)
-	(wire
-		(pts
 			(xy 176.53 72.39) (xy 177.8 72.39)
 		)
@@
 	(wire
 		(pts
+			(xy 133.35 77.47) (xy 135.89 77.47)
+		)
+		(stroke
+			(width 0)
+			(type default)
+		)
+	)
+	(wire
+		(pts
 			(xy 153.67 36.83) (xy 153.67 39.37)
 		)
@@
 		(pts
 			(xy 156.21 125.73) (xy 156.21 128.27)
+		)
+		(stroke
+			(width 0)
+			(type default)
+		)
+	)
+	(wire
+		(pts
+			(xy 133.35 74.93) (xy 135.89 74.93)
 		)
 		(stroke
@@
 	)
 	(label "THERM2_ADC"
-		(at 190.5 62.23 180)
+		(at 190.5 87.63 180)
 		(effects
 			(font
@@
 	)
 	(label "THERM1_ADC"
-		(at 190.5 87.63 180)
+		(at 190.5 62.23 180)
 		(effects
 			(font
@@
 	(hierarchical_label "GPS_RST"
 		(shape output)
-		(at 132.08 82.55 180)
+		(at 133.35 74.93 180)
 		(effects
 			(font
@@
 	(hierarchical_label "GPS_TP"
 		(shape input)
-		(at 177.8 64.77 0)
-		(effects
-			(font
-				(size 1.27 1.27)
-			)
-			(justify left)
-		)
-	)
+		(at 133.35 77.47 180)
+		(effects
+			(font
+				(size 1.27 1.27)
+			)
+			(justify right)
+		)
+	)
