File: telem_mcu.kicad_sch (KiCad schematic)
At the start: 28 parts, among them J3 Conn_01x06, J5 Micro_SD_Card, SW2 SW_Push, U3 STM32F373CCTx, X1 32.768kHz

Commit message: Updated Schematics & finished rev2 layout. Routing left
Parts:
- removed C11, C12, C17, C18, C20, C5, C7, C9: 100nF, Capacitor_SMD:C_0603_1608Metric, symbol Device:C
- added C31, C32, C33, C34, C35, C36, C37, C38: 100nF, Capacitor_SMD:C_0603_1608Metric, symbol Device:C
- C10, C15, C16, C6, C8: Voltage Rating (none) -> 10V
Connections:
- net +3V3: now also C34.1, C35.1, C36.1, C37.1, C38.1
- net PGND: now also C31.2, C32.2, C33.1, C34.2, C35.2, C36.2, C37.2, C38.2
- net RESET: now also C33.2
- net THERM1_ADC: now also C31.1
- net THERM2_ADC: now also C32.1
