File: telem_sensors.kicad_sch (KiCad schematic)
At the start: 29 parts, among them J4 Thermistor Molex, J6 Thermistor Molex, J8 SMA, U10 MAX-M10S, U4 LSM6DSRXTR, U5 MCP6L01x-xLT, U7 BMP585, U8 MCP6L01x-xLT

Commit message: Updated schematics for rev2
Parts:
- C21, C26, C27, C32, C33: footprint Capacitor_SMD:C_0805_2012Metric -> Capacitor_SMD:C_0603_1608Metric
Connections:
- net IMU_INT: no longer names the net of U4.4 (INT1)
- no-connect marks 8 -> 9
Changed lines of the file:
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@@
 	)
 	(no_connect
+		(at 71.12 95.25)
+	)
+	(no_connect
 		(at 177.8 106.68)
 	)
@@
 		)
 	)
-	(hierarchical_label "IMU_INT"
-		(shape output)
-		(at 71.12 95.25 180)
-		(effects
-			(font
-				(size 1.27 1.27)
-			)
-			(justify right)
-		)
-	)
 	(hierarchical_label "IMU_SPC"
 		(shape input)
@@
 			)
 		)
-		(property "Footprint" "Capacitor_SMD:C_0805_2012Metric"
+		(property "Footprint" "Capacitor_SMD:C_0603_1608Metric"
 			(at 129.2352 110.49 0)
 			(hide yes)
@@
 			)
 		)
-		(property "Footprint" "Capacitor_SMD:C_0805_2012Metric"
+		(property "Footprint" "Capacitor_SMD:C_0603_1608Metric"
 			(at 174.9552 99.06 0)
 			(hide yes)
@@
 			)
 		)
-		(property "Footprint" "Capacitor_SMD:C_0805_2012Metric"
+		(property "Footprint" "Capacitor_SMD:C_0603_1608Metric"
 			(at 63.1952 148.59 0)
 			(hide yes)
@@
 			)
 		)
-		(property "Footprint" "Capacitor_SMD:C_0805_2012Metric"
+		(property "Footprint" "Capacitor_SMD:C_0603_1608Metric"
 			(at 125.4252 143.51 0)
 			(hide yes)
@@
 			)
 		)
-		(property "Footprint" "Capacitor_SMD:C_0805_2012Metric"
+		(property "Footprint" "Capacitor_SMD:C_0603_1608Metric"
 			(at 214.3252 99.06 0)
 			(hide yes)

Commit message: Initial Layout Rev2
Connections:
- net PGND: now also J4.1 (Pin_1); no longer J4.2 (Pin_2)
- net THERM1_V-: now also J4.2 (Pin_2); no longer J4.1 (Pin_1)
Other:
- moved on the sheet: J4
Changed lines of the file:
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@@
+	)
+	(junction
+		(at 173.99 48.26)
+		(diameter 0)
+		(color 0 0 0 0)
 	)
 	(junction
@@
 	)
 	(junction
-		(at 173.99 48.26)
-		(diameter 0)
-		(color 0 0 0 0)
-	)
-	(junction
 		(at 52.07 92.71)
 		(diameter 0)
@@
 	)
 	(junction
-		(at 73.66 50.8)
-		(diameter 0)
-		(color 0 0 0 0)
-	)
-	(junction
 		(at 133.35 50.8)
 		(diameter 0)
@@
 		(color 0 0 0 0)
 	)
+	(junction
+		(at 73.66 50.8)
+		(diameter 0)
+		(color 0 0 0 0)
+	)
 	(no_connect
 		(at 177.8 104.14)
@@
 	(wire
 		(pts
+			(xy 173.99 55.88) (xy 173.99 63.5)
+		)
+		(stroke
+			(width 0)
+			(type default)
+		)
+	)
+	(wire
+		(pts
 			(xy 118.11 135.89) (xy 124.46 135.89)
 		)
@@
 		(pts
 			(xy 58.42 97.79) (xy 71.12 97.79)
-		)
-		(stroke
-			(width 0)
-			(type default)
-		)
-	)
-	(wire
-		(pts
-			(xy 173.99 55.88) (xy 173.99 63.5)
 		)
 		(stroke
@@
 	(symbol
 		(lib_id "Connector_Generic:Conn_01x02")
-		(at 68.58 55.88 0)
-		(mirror y)
+		(at 68.58 58.42 180)
 		(unit 1)
 		(body_style 1)
@@
 		(dnp no)
 		(property "Reference" "J4"
-			(at 57.404 59.69 0)
+			(at 57.404 54.61 0)
 			(show_name no)
 			(do_not_autoplace no)
@@
 		)
 		(property "Footprint" "Connector_Molex:Molex_MicroClasp_55935-0230_1x02_P2.00mm_Horizontal"
-			(at 68.58 55.88 0)
+			(at 68.58 58.42 0)
 			(hide yes)
 			(show_name no)
@@
 		)
 		(property "Datasheet" ""
-			(at 68.58 55.88 0)
+			(at 68.58 58.42 0)
 			(hide yes)
 			(show_name no)
@@
 		)
 		(property "Description" "Generic connector, single row, 01x02, script generated (kicad-library-utils/schlib/autogen/connector/)"
-			(at 68.58 55.88 0)
-			(hide yes)
-			(show_name no)
+			(at 68.58 58.42 0)
+			(hide yes)
+			(show_name no)
